Commit message: depth cam dadded(ASUS)

File: simple_hexapod_description/urdf/simple_hexapod.urdf (robot description, URDF)
Before this commit: robot Simple_Hexapod, 32 links, 31 joints
Links:
- added link depth_camera_depth_frame
- added link depth_camera_depth_optical_frame
- added link depth_camera_link, mass 0.200; collision box size=0.035 0.185 0.025; visual mesh filename=package://hector_sensors_description/meshes/asus_camera/asu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
- added link depth_camera_rgb_frame
- added link depth_camera_rgb_optical_frame
Joints:
- added joint depth_camera_depth_joint: type fixed, parent depth_camera_link, child depth_camera_depth_frame, origin xyz=0.0 0.049 0.0 rpy=0 0 0
- added joint depth_camera_depth_optical_joint: type fixed, parent depth_camera_depth_frame, child depth_camera_depth_optical_frame, origin xyz=0 0 0 rpy=-1.57079632679 0.0 -1.57079632679
- added joint depth_camera_joint: type fixed, parent base_link, child depth_camera_link, origin xyz=0.125 0 0.04 rpy=0 0 0
- added joint depth_camera_rgb_joint: type fixed, parent depth_camera_link, child depth_camera_rgb_frame, origin xyz=0.0 0.022 0.0 rpy=0 0 0
- added joint depth_camera_rgb_optical_joint: type fixed, parent depth_camera_rgb_frame, child depth_camera_rgb_optical_frame, origin xyz=0 0 0 rpy=-1.57079632679 0.0 -1.57079632679

File: simple_hexapod_description/urdf/simple_hexapod.xacro (robot description, xacro)
@@ -2,12 +2,19 @@
 <robot name="Simple_Hexapod"  xmlns:xacro="http://www.ros.org/wiki/xacro">
   <xacro:include filename="$(find simple_hexapod_description)/urdf/simple_hexapod_urdf.xacro" />
+  <xacro:include filename="$(find simple_hexapod_description)/urdf/asus_camera.urdf.xacro" />
   <link name="base_link"/>
-    <xacro:simple_hexapod parent="base_link">
+	<xacro:simple_hexapod parent="base_link">
         <origin xyz="0 0 0" rpy="0 0 0" />
     </xacro:simple_hexapod>
-  <gazebo>
-    <plugin filename="libgazebo_ros_control.so" name="gazebo_ros_control">
-      <robotNamespace>/simple_hexapod</robotNamespace>
-    </plugin>
-  </gazebo>
+	<!--<xacro:camera parent="base_link">
+        <origin xyz="0 0 1" rpy="0 0 0" />
+    </xacro:camera>-->
+	<xacro:asus_camera name="depth_camera" parent="base_link">
+    	<origin xyz="0.125 0 0.04" rpy="0 0 0"/>
+  	</xacro:asus_camera>
+	<gazebo>
+    	<plugin filename="libgazebo_ros_control.so" name="gazebo_ros_control">
+      	<robotNamespace>/simple_hexapod</robotNamespace>
+    	</plugin>
+  	</gazebo>
 </robot>

File: simple_hexapod_description/urdf/simple_hexapod_urdf.xacro (robot description, xacro)
@@ -5,4 +5,5 @@
 <xacro:property name="thigh_offset_y" value="-0.0645" />
 <xacro:property name="thigh_offset_z" value="-0.0145" />
+<xacro:property name="camera_link" value="0.05" /> <!-- Size of square 'camera' box -->
 <xacro:macro name="simple_hexapod" params="parent *origin">
       <joint name="j_simple_hexapod_attachment" type="fixed">
