Commit message: lms1xx laser added

File: simple_hexapod_description/urdf/simple_hexapod.xacro (robot description, xacro)
@@ -2,5 +2,6 @@
 <robot name="Simple_Hexapod"  xmlns:xacro="http://www.ros.org/wiki/xacro">
   <xacro:include filename="$(find simple_hexapod_description)/urdf/simple_hexapod_urdf.xacro" />
-  <xacro:include filename="$(find simple_hexapod_description)/urdf/asus_camera.urdf.xacro" />
+  <xacro:include filename="$(find simple_hexapod_description)/urdf/sensor_urdf/asus_camera.urdf.xacro" />
+  <xacro:include filename="$(find simple_hexapod_description)/urdf/sensor_urdf/sick_lms1xx_mount.urdf.xacro" />
   <link name="base_link"/>
 	<xacro:simple_hexapod parent="base_link">
@@ -13,4 +14,7 @@
     	<origin xyz="0.125 0 0.04" rpy="0 0 0"/>
   	</xacro:asus_camera>
+	<xacro:sick_lms1xx_mount parent="base_link">
+    	<origin xyz="0 0 0.0175" rpy="0 0 0"/>
+  	</xacro:sick_lms1xx_mount>
 	<gazebo>
     	<plugin filename="libgazebo_ros_control.so" name="gazebo_ros_control">
